Commit message: Add camera sensor

File: urdf/udacity_bot.xacro (robot description, xacro)
@@ -23,4 +23,32 @@
     <joint_properties damping="1.0" friction="1.0"/>
   </joint>
+  <joint type="fixed" name="camera_joint">
+    <origin xyz="0.2 0 0" rpy="0 0 0"/>
+    <child link="camera"/>
+    <parent link="chassis"/>
+  </joint>
+  <link name="camera">
+    <inertial>
+      <mass value="0.1"/>
+      <origin xyz="0 0 0" rpy="0 0 0"/>
+      <inertia
+              ixx="1e-6" ixy="0" ixz="0"
+              iyy="1e-6" iyz="0"
+              izz="1e-6"
+      />
+    </inertial>
+    <collision name='camera_collision'>
+      <origin xyz="0 0 0" rpy="0 0 0"/>
+      <geometry>
+        <box size="0.05 0.05 0.05"/>
+      </geometry>
+    </collision>
+    <visual name='camera_visual'>
+      <origin xyz="0 0 0" rpy="0 0 0"/>
+      <geometry>
+        <box size="0.05 0.05 0.05"/>
+      </geometry>
+    </visual>
+  </link>
   <link name="left_wheel">
     <inertial>

Commit message: Add Laser Rangefinder

File: urdf/udacity_bot.xacro (robot description, xacro)
@@ -28,4 +28,32 @@
     <parent link="chassis"/>
   </joint>
+  <joint type="fixed" name="hokuyo_joint">
+    <origin xyz=".15 0 .1" rpy="0 0 0"/>
+    <child link="hokuyo"/>
+    <parent link="chassis"/>
+  </joint>
+  <link name="hokuyo">
+    <inertial>
+      <mass value="0.1"/>
+      <origin xyz="0 0 0" rpy="0 0 0"/>
+      <inertia
+              ixx="1e-6" ixy="0" ixz="0"
+              iyy="1e-6" iyz="0"
+              izz="1e-6"
+      />
+    </inertial>
+    <collision name='hokuyo_collision'>
+      <origin xyz="0 0 0" rpy="0 0 0"/>
+      <geometry>
+        <box size="0.1 0.1 0.1"/>
+      </geometry>
+    </collision>
+    <visual name='hokuyo_visual'>
+      <origin xyz="0 0 0" rpy="0 0 0"/>
+      <geometry>
+        <mesh filename="package://udacity_bot/meshes/hokuyo.dae"/>
+      </geometry>
+    </visual>
+  </link>
   <link name="camera">
     <inertial>

Commit message: Fix RViz robot colors

File: urdf/udacity_bot.xacro (robot description, xacro)
@@ -1,4 +1,10 @@
 <?xml version='1.0'?>
 <robot name="udacity_bot" xmlns:xacro="http://www.ros.org/wiki/xacro">
+  <material name="Blue">
+    <color rgba="0.0 0.0 0.8 1.0"/>
+  </material>
+  <material name="Red">
+    <color rgba="0.8 0.0 0.0 1.0"/>
+  </material>
   <xacro:include filename="$(find udacity_bot)/urdf/udacity_bot.gazebo" />
   <link name="robot_footprint"></link>
@@ -101,4 +107,5 @@
         <cylinder radius="0.1" length="0.05"/>
       </geometry>
+      <material name="Red"/>
     </visual>
   </link>
@@ -124,4 +131,5 @@
         <cylinder radius="0.1" length="0.05"/>
       </geometry>
+      <material name="Red"/>
     </visual>
   </link>
@@ -148,4 +156,5 @@
         <box size=".4 .2 .1"/>
       </geometry>
+      <material name="Blue"/>
     </visual>
     <collision name='back_caster_collision'>
