Commit message: Fix custom bot

File: urdf/custom_bot.xacro (robot description, xacro)
@@ -47,5 +47,5 @@
   </joint>
   <joint type="fixed" name="hokuyo_joint">
-    <origin xyz=".15 0 .175" rpy="0 0 0"/>
+    <origin xyz=".15 0 .2" rpy="0 0 0"/>
     <child link="hokuyo"/>
     <parent link="tower"/>
@@ -173,5 +173,5 @@
     <pose>0 0 0.1 0 0 0</pose>
     <inertial>
-      <mass value="15.0"/>
+      <mass value="10.0"/>
       <origin xyz="0.0 0 0" rpy=" 0 0 0"/>
       <inertia
